File: hardware/IntelliThings.kicad_pcb (KiCad board)
At the start: 2 copper layers, 140 x 80 mm, 7 parts, among them J1 USB_C_Receptacle_PowerOnly_6P, U1 ESP32-C6-DevKitC-1

Commit message: NEW FILES for 10/25
Parts:
- added J2: SGP40, IntelliThings:SGP40 Footprint, F.Cu at (163.6, 59.1)
- added J3: BH1750, Connector_PinHeader_2.54mm:PinHeader_1x06_P2.54mm_Vertical, F.Cu at (166.9, 112.0)
- added J4: VL53L0X, Connector_PinHeader_2.54mm:PinHeader_1x06_P2.54mm_Vertical, F.Cu at (146.4, 112.0)
- added J5: SCD41, IntelliThings:SCD41 Footprint, F.Cu at (184.9, 88.5)
- added J6: SHT41, IntelliThings:SHT41 Footprint, F.Cu at (163.5, 88.9)
- moved J1 3.89 mm to (152.5, 60.6)
