File: hardware/IntelliThings.kicad_sch (KiCad schematic)
At the start: 12 parts, among them J1 USB_C_Receptacle_PowerOnly_6P, J2 SGP40, J3 BH1750, J4 VL53L0X, J5 SCD41, J6 SHT41, U1 ESP32-C6-DevKitC-1

Commit message: NEW FILES for 10/25
Parts:
- added J7: PM2.5, Connector_PinHeader_2.54mm:PinHeader_1x08_P2.54mm_Vertical, symbol Connector:Conn_01x08_Socket
- J2: footprint (none) -> IntelliThings:SGP40 Footprint
- J3, J4: footprint (none) -> Connector_PinHeader_2.54mm:PinHeader_1x06_P2.54mm_Vertical
- J5: footprint (none) -> IntelliThings:SCD41 Footprint
- J6: footprint (none) -> IntelliThings:SHT41 Footprint
Connections:
- net +5V: now also J7.8 (Pin_8)
- net GND: now also J7.7 (Pin_7)
- net LPRX: now reaches U1.3 (GPIO4/MTMS)
- net LPRX: now also J7.5 (Pin_5)
- net LPTX: now reaches U1.4 (GPIO5/MTDI)
- net LPTX: now also J7.4 (Pin_4)
- no-connect marks 9 -> 13
Other:
- note added: "UART CONNECTION - SCREEN"
- note added: "UART SENSORS"
- note removed: "Custom footprints will be required for each of these sensors"
